File: termokip/termokip.kicad_sch (KiCad schematic)
At the start: 0 parts

Commit message: Iniciando o desenvolvimento do esquematico reaproveitando partes já validadas na versão anterior.
Parts:
- added AE1: Antenna_Shield, RF_Antenna:Texas_SWRA117D_2.4GHz_Right, symbol Device:Antenna_Shield
- added C1: 100n, Capacitor_SMD:C_0603_1608Metric, symbol Device:C
- added C10: 1.0pF, Capacitor_SMD:C_0603_1608Metric, symbol Device:C
- added C2: 4.7u, Capacitor_SMD:C_0603_1608Metric, symbol Device:C
- added C3, C4: NC, Capacitor_SMD:C_0603_1608Metric, symbol Device:C
- added C5, C7: 18pF, Capacitor_SMD:C_0603_1608Metric, symbol Device:C
- added C6, C8: 1uF, symbol Device:C
- added C9: 1.2pF, Capacitor_SMD:C_0603_1608Metric, symbol Device:C
- added D1: BAT760, BAT_760:SOD323_F_, symbol BAT_760:BAT760
- added J1: USB_B, USB_B:CUI_UJ2-BV-1-TH, symbol Connector:USB_B
- added J2: Screw_Terminal_01x08, TerminalBlock:TerminalBlock_MaiXu_MX126-5.0-08P_1x08_P5.00mm, symbol Connector:Screw_Terminal_01x08
- added L1: 2.7nH, Inductor_SMD:L_0805_2012Metric, symbol Device:L
- added R1, R2, R3, R4, R5, R6, R7, R8: 0Ω, Resistor_SMD:R_0603_1608Metric, symbol Device:R
- added U1: USBLC6-2SC6, Package_TO_SOT_SMD:SOT-23-6, symbol Power_Protection:USBLC6-2SC6
- added U2: W25Q128JVSIQ, MEMORIA_FLESH:SOIC127P790X216-8N, symbol MEMORIA_FLESH:W25Q128JVSIQ
- added U3: AP2112K-3.3, Package_TO_SOT_SMD:SOT-23-5, symbol Regulator_Linear:AP2112K-3.3
- added U4: ESP32-S3, Package_DFN_QFN:QFN-56-1EP_7x7mm_P0.4mm_EP4x4mm, symbol MCU_Espressif:ESP32-S3
- added X1: OSCILADOR-3225, OSCILADOR_3225:TSX-3225, symbol OSCILADOR_3225:TSX-3225
Connections:
- new net: C1.1, C2.1, D1.2, J1.1 (VBUS), U1.5 (VBUS)
- new net: R2.2, U2.5 (DI(IO0))
- new net: C4.1, R6.2, U1.1 (I/O1)
- new net: C3.1, R7.1, U1.3 (I/O2)
- new net: C5.1, R8.1, X1.1
- new net: R4.2, U2.3 (/WP(IO2))
- new net: R5.2, U2.7 (/HOLD/RESET(IO3))
- new net: R1.2, U2.6 (CLK)
- new net: J1.2 (D-), R7.2
- new net: J1.3 (D+), R6.1
- new net: AE1.1 (A), C10.1, L1.2
- new net: U4.2 (VDD3P3), U4.3 (VDD3P3)
- new net: U4.55 (VDDA), U4.56 (VDDA)
- new net: R3.2, U2.2 (DO(IO1))
- new net AU_LORA: J2.8 (Pin_8), U4.27 (GPIO21)
- new net BOOT: U4.5 (GPIO0)
- new net D+: U1.6 (I/O1), U4.26 (GPIO20/USB_D+)
- new net D-: U1.4 (I/O2), U4.25 (GPIO19/USB_D-)
- new net DATA_LED: U4.9 (GPIO4)
- new net EN: U4.4 (CHIP_PU)
- new net GND: AE1.2 (Shield), C1.2, C10.2, C2.2, C3.2, C4.2, C5.2, C6.2, C7.2, C8.2, C9.2, J1.4 (GND), J1.5 (Shield), J2.3 (Pin_3), U1.2 (GND), U2.4 (GND), U3.2 (GND), U4.57 (GND), X1.2, X1.4
- new net GPIO1: U4.6 (GPIO1)
- new net GPIO2: U4.7 (GPIO2)
- new net GPIO45: U4.51 (GPIO45)
- new net GPIO5: U4.10 (GPIO5)
- new net LINE_3.3: C8.1, U3.5 (VOUT)
- new net LNA_IN: C9.1, L1.1, U4.1 (LNA_IN)
- new net M0_LORA: J2.6 (Pin_6), U4.38 (GPIO33)
- new net M1_LORA: J2.7 (Pin_7), U4.39 (GPIO34)
- new net M_TXD0: U4.49 (U0TXD)
- new net RX_LORA: J2.5 (Pin_5), U4.24 (GPIO18)
- new net SPICLK: R1.1, U4.33 (SPICLK)
- new net SPICS0: U2.1 (/CS), U4.32 (SPICS0)
- new net SPID: R2.1, U4.35 (SPID)
- new net SPIHD: R5.1, U4.30 (SPIHD)
- new net SPIQ: R3.1, U4.34 (SPIQ)
- new net SPIWP: R4.1, U4.31 (SPIWP)
- new net TX_LORA: J2.4 (Pin_4), U4.23 (GPIO17)
- new net VDD_SPI: U2.8 (VCC), U4.29 (VDD_SPI)
- new net VIN_5V: C6.1, D1.1, J2.1 (Pin_1), U3.1 (VIN), U3.3 (EN)
- new net XTAL_N: C7.1, U4.53 (XTAL_N), X1.3
- new net XTAL_P: R8.2, U4.54 (XTAL_P)
- no-connect marks 0 -> 25
Other:
- note added: "ANTENA WI-FI"
- note added: "ESTABILIZADOR 3.3"
- note added: "INPUT USB"
- note added: "MCU"
- note added: "MEMORIA_FLASH"
- note added: "TERMINAIS"
- note added: "U3 NC"
- note added: "XTAL"
