File: termokip/projeto_eletronico/termokip/termokip.kicad_sch (KiCad schematic)
At the start: 0 parts

Commit message: Iniciando o desenvolvimento do esquematico
Parts:
- added C1: 100n, Capacitor_SMD:C_0603_1608Metric, symbol Device:C
- added C2: 4.7u, Capacitor_SMD:C_0603_1608Metric, symbol Device:C
- added C3, C4: NC, Capacitor_SMD:C_0603_1608Metric, symbol Device:C
- added C5, C6: 1uF, symbol Device:C
- added D1: BAT760, BAT_760:SOD323_F_, symbol BAT_760:BAT760
- added J1: USB_B, USB_B:CUI_UJ2-BV-1-TH, symbol Connector:USB_B
- added R1, R2: 0Ω, Resistor_SMD:R_0603_1608Metric, symbol Device:R
- added R8: 10k, symbol Device:R
- added U1: USBLC6-2SC6, Package_TO_SOT_SMD:SOT-23-6, symbol Power_Protection:USBLC6-2SC6
- added U2: CH32V003FxPx, Package_SO:TSSOP-20_4.4x6.5mm_P0.65mm, symbol MCU_WCH_CH32V0:CH32V003FxPx
- added U3: AP2112K-3.3, Package_TO_SOT_SMD:SOT-23-5, symbol Regulator_Linear:AP2112K-3.3
- added U6: TMP117xxDRV, Package_SON:WSON-6-1EP_2x2mm_P0.65mm_EP1x1.6mm, symbol Sensor_Temperature:TMP117xxDRV
Connections:
- new net: C1.1, C2.1, D1.2, J1.1 (VBUS), U1.5 (VBUS)
- new net: R8.2, U6.4 (ADD0)
- new net: C4.1, R1.2, U1.1 (I/O1)
- new net: C3.1, R2.1, U1.3 (I/O2)
- new net: J1.2 (D-), R2.2
- new net: J1.3 (D+), R1.1
- new net D+: U1.6 (I/O1)
- new net D-: U1.4 (I/O2)
- new net GND: C1.2, C2.2, C3.2, C4.2, C5.2, C6.2, J1.4 (GND), J1.5 (Shield), R8.1, U1.2 (GND), U3.2 (GND), U6.2 (GND)
- new net LINE_3.3: C6.1, U3.5 (VOUT)
- new net MP_OUTPUT: C5.1, U3.1 (VIN), U3.3 (EN)
- new net TMP_ALERT: U6.3 (ALERT)
- new net TMP_SCL: U6.1 (SCL)
- new net TMP_SDA: U6.6 (SDA)
- new net VDD_3.3_TMP: U6.5 (V+)
- new net VIN_5V: D1.1
Other:
- note added: "ESTABILIZADOR 3.3"
- note added: "INPUT USB"
- note added: "SENS_TEMP"
